Commit message: Fixed bug in the mesh loading

File: xacro/depthCamera.xacro (robot description, xacro)
@@ -17,5 +17,5 @@
             <origin xyz="0 0 0" rpy="0 0 0"/>
             <geometry>
-                <mesh filename="package://go1_description/meshes/depthCamera.dae" scale="1 1 1"/>
+                <mesh filename="file://$(find go1_description)/meshes/depthCamera.dae" scale="1 1 1"/>
             </geometry>
             </visual>
