Commit message: ros2 pkg

File: xacro/robot.xacro (robot description, xacro)
@@ -7,6 +7,6 @@
     <!-- <xacro:include filename="$(find go1_description)/xacro/stairs.xacro"/> -->
     <xacro:include filename="$(find go1_description)/xacro/gazebo.xacro"/>
-    <xacro:include filename="$(find go1_description)/xacro/depthCamera.xacro"/>
-    <xacro:include filename="$(find go1_description)/xacro/ultraSound.xacro"/>
+    <!-- <xacro:include filename="$(find go1_description)/xacro/depthCamera.xacro"/>
+    <xacro:include filename="$(find go1_description)/xacro/ultraSound.xacro"/> -->
     <!-- <xacro:include filename="$(find go1_gazebo)/launch/stairs.urdf.xacro"/> -->
     <!-- <xacro:stairs stairs="15" xpos="0" ypos="0" zpos="0" /> -->
@@ -39,5 +39,5 @@
             <origin rpy="0 0 0" xyz="0 0 0"/>
             <geometry>
-                <mesh filename="package://go1_description/meshes/trunk.dae" scale="1 1 1"/>
+                <mesh filename="file://$(find go1_description)/meshes/trunk.dae" scale="1 1 1"/>
             </geometry>
             <!-- <material name="orange"/> -->
@@ -87,5 +87,5 @@
     <xacro:leg name="RR" mirror="-1" mirror_dae="False"  front_hind="-1" front_hind_dae="False" />
     <xacro:leg name="RL" mirror="1"  mirror_dae="True"   front_hind="-1" front_hind_dae="False" />
-    <xacro:depthCamera camID="1" name="face">
+    <!-- <xacro:depthCamera camID="1" name="face">
         <origin rpy="${PI} 0 0" xyz="0.2785 0.0125 0.0167"/>
     </xacro:depthCamera>
@@ -124,4 +124,4 @@
     <xacro:ultraSound name="face">
         <origin rpy="0 0 0" xyz="0.2747 0.0 -0.0088"/>
-    </xacro:ultraSound>
+    </xacro:ultraSound> -->
 </robot>

Commit message: Added a check for the ROS version so that the plugins work for either ROS 1 or ROS 2

File: xacro/gazebo.xacro (robot description, xacro)
@@ -1,45 +1,46 @@
 <?xml version="1.0"?>
-<robot>
+<robot xmlns:xacro="http://www.ros.org/wiki/xacro">
+    <!-- Define the ROS version as a property -->
+    <xacro:property name="ros_version" value="$(env ROS_VERSION)" />
     <!-- ros_control plugin -->
-    <!-- <gazebo>
-        <plugin name="gazebo_ros_control" filename="libgazebo_ros_control.so">
-            <robotNamespace>/go1_gazebo</robotNamespace>
-            <robotSimType>gazebo_ros_control/DefaultRobotHWSim</robotSimType>
-        </plugin>
-    </gazebo> -->
-    <!-- <gazebo>
-        <plugin filename="libgazebo_ros2_control.so" name="gazebo_ros2_control">
-        <parameters>"file://$(find go1_description)/config/ros_control/ros_control.yaml</parameters>
-      </plugin>
-    </gazebo> -->
     <gazebo>
-        <plugin filename="libgazebo_ros2_control.so" name="gazebo_ros2_control">
-        <parameters>$(find go1_description)/config/ros_control/ros_control.yaml</parameters>
-      </plugin>
+        <xacro:if value="${ros_version == 1}">
+            <plugin name="gazebo_ros_control" filename="libgazebo_ros_control.so">
+                <robotNamespace>/go1_gazebo</robotNamespace>
+                <robotSimType>gazebo_ros_control/DefaultRobotHWSim</robotSimType>
+            </plugin>
+        </xacro:if>
+        <xacro:if value="${ros_version == 2}">
+            <plugin filename="libgazebo_ros2_control.so" name="gazebo_ros2_control">
+            <parameters>$(find go1_description)/config/ros_control/ros_control.yaml</parameters>
+          </plugin>
+        </xacro:if>
     </gazebo>
     <!-- Show the trajectory of trunk center. -->
-    <!-- <gazebo>
-        <plugin name="3dplot" filename="libLinkPlot3DPlugin.so">
-            <frequency>10</frequency>
-            <plot>
-                <link>base</link>
-                <pose>0 0 0 0 0 0</pose>
-                <material>Gazebo/Yellow</material>
-            </plot>
-        </plugin>
-    </gazebo> -->
     <gazebo>
-        <plugin name="p3d_base_controller" filename="libgazebo_ros_p3d.so">
-          <ros>
-              <argument>odom:=odom/ground_truth</argument>
-          </ros>
-          <body_name>base</body_name>
-          <frame_name>world</frame_name>
-          <update_rate>10.0</update_rate>
-          <xyz_offset>0 0 0</xyz_offset>
-          <rpy_offset>0 0 0</rpy_offset>
-          <gaussian_noise>0.01</gaussian_noise>
-      </plugin>
-      </gazebo>
+        <xacro:if value="${ros_version == 1}">
+            <plugin name="3dplot" filename="libLinkPlot3DPlugin.so">
+                <frequency>10</frequency>
+                <plot>
+                    <link>base</link>
+                    <pose>0 0 0 0 0 0</pose>
+                    <material>Gazebo/Yellow</material>
+                </plot>
+            </plugin>
+        </xacro:if>
+        <xacro:if value="${ros_version == 2}">
+            <plugin name="p3d_base_controller" filename="libgazebo_ros_p3d.so">
+              <ros>
+                  <argument>odom:=odom/ground_truth</argument>
+              </ros>
+              <body_name>base</body_name>
+              <frame_name>world</frame_name>
+              <update_rate>10.0</update_rate>
+              <xyz_offset>0 0 0</xyz_offset>
+              <rpy_offset>0 0 0</rpy_offset>
+              <gaussian_noise>0.01</gaussian_noise>
+          </plugin>
+        </xacro:if>
+    </gazebo>
     <!-- Show the trajectory of foot. You can add another trajectory about another foot. -->
     <!-- <gazebo>
@@ -53,11 +54,19 @@
         </plugin>
     </gazebo> -->
-    <!-- <gazebo>
-        <plugin filename="libgazebo_ros_force.so" name="gazebo_ros_force">
-            <bodyName>trunk</bodyName>
-            <topicName>/apply_force/trunk</topicName>
-        </plugin>
-    </gazebo> -->
-    <!-- <gazebo reference="imu_link">
+    <gazebo>
+        <xacro:if value="${ros_version == 1}">
+            <plugin filename="libgazebo_ros_force.so" name="gazebo_ros_force">
+                <bodyName>trunk</bodyName>
+                <topicName>/apply_force/trunk</topicName>
+            </plugin>
+        </xacro:if>
+        <xacro:if value="${ros_version == 2}">
+            <plugin filename="libgazebo_ros_force.so" name="gazebo_ros_force">
+                <link_name>base</link_name>
+                <topicName>/apply_force/trunk</topicName>
+            </plugin>
+        </xacro:if>
+    </gazebo>
+    <gazebo reference="imu_link">
         <gravity>true</gravity>
         <sensor name="imu_sensor" type="imu">
@@ -76,25 +85,4 @@
             </plugin>
             <pose>0 0 0 0 0 0</pose>
-        </sensor>
-    </gazebo> -->
-    <gazebo reference="imu_link">
-        <sensor name="imu_controller" type="imu">
-            <always_on>true</always_on>
-            <update_rate>50</update_rate>
-            <plugin name="gazebo_ros_imu_sensor" filename="libgazebo_ros_imu_sensor.so">
-                <ros>
-                    <namespace>/imu</namespace>
-                    <argument>~/out:=data</argument>
-                </ros>
-                <!-- <updateRate>50.0</updateRate>
-                <bodyName>imu_link</bodyName>
-                <topicName>imu/data</topicName>
-                <accelDrift>0.005 0.005 0.005</accelDrift>
-                <accelGaussianNoise>0.005 0.005 0.005</accelGaussianNoise>
-                <rateDrift>0.005 0.005 0.005 </rateDrift>
-                <rateGaussianNoise>0.005 0.005 0.005 </rateGaussianNoise>
-                <headingDrift>0.005</headingDrift>
-                <headingGaussianNoise>0.005</headingGaussianNoise> -->
-            </plugin>
         </sensor>
     </gazebo>
@@ -170,5 +158,5 @@
         </sensor>
     </gazebo> -->
-  <!-- <gazebo reference="depthCamera_link_left">
+  <gazebo reference="depthCamera_link_left">
     <sensor name="camera_link_camera" type="depth">
       <update_rate>20</update_rate>
@@ -210,7 +198,7 @@
       </plugin>
     </sensor>
-  </gazebo> -->
+  </gazebo>
     <!-- Foot contacts. -->
-    <!-- <gazebo reference="FR_calf">
+    <gazebo reference="FR_calf">
         <sensor name="FR_foot_contact" type="contact">
         <update_rate>100</update_rate>
@@ -247,7 +235,7 @@
         </contact>
         </sensor>
-    </gazebo> -->
+    </gazebo>
     <!-- Visualization of Foot contacts. -->
-    <!-- <gazebo reference="FR_foot">
+    <gazebo reference="FR_foot">
         <visual>
             <plugin name="drawForcePlugin" filename="libunitreeDrawForcePlugin.so">
@@ -276,5 +264,5 @@
             </plugin>
         </visual>
-    </gazebo> -->
+    </gazebo>
     <gazebo reference="base">
         <material>Gazebo/Green</material>

File: xacro/leg.xacro (robot description, xacro)
@@ -251,29 +251,32 @@
         </link>
         <xacro:leg_transmission name="${name}"/>
-        <ros2_control name="${name}" type="system">
-            <hardware>
-                <plugin>gazebo_ros2_control/GazeboSystem</plugin>
-            </hardware>
-            <joint name="${name}_hip_joint">
-                <command_interface name="effort"/>
-                <state_interface name="position"/>
-                <state_interface name="velocity"/>
-            </joint>
-            <joint name="${name}_thigh_joint">
-                <command_interface name="effort"/>
-                <state_interface name="position"/>
-                <state_interface name="velocity"/>
-            </joint>
-            <joint name="${name}_calf_joint">
-                <command_interface name="effort"/>
-                <state_interface name="position"/>
-                <state_interface name="velocity"/>
-            </joint>
-            <joint name="${name}_foot_fixed">
-                <command_interface name="effort"/>
-                <state_interface name="position"/>
-                <state_interface name="velocity"/>
-            </joint>
-        </ros2_control>
+        <xacro:property name="ros_version" value="$(env ROS_VERSION)" />
+        <xacro:if value="${ros_version == 2}">
+            <ros2_control name="${name}" type="system">
+                <hardware>
+                    <plugin>gazebo_ros2_control/GazeboSystem</plugin>
+                </hardware>
+                <joint name="${name}_hip_joint">
+                    <command_interface name="effort"/>
+                    <state_interface name="position"/>
+                    <state_interface name="velocity"/>
+                </joint>
+                <joint name="${name}_thigh_joint">
+                    <command_interface name="effort"/>
+                    <state_interface name="position"/>
+                    <state_interface name="velocity"/>
+                </joint>
+                <joint name="${name}_calf_joint">
+                    <command_interface name="effort"/>
+                    <state_interface name="position"/>
+                    <state_interface name="velocity"/>
+                </joint>
+                <joint name="${name}_foot_fixed">
+                    <command_interface name="effort"/>
+                    <state_interface name="position"/>
+                    <state_interface name="velocity"/>
+                </joint>
+            </ros2_control>
+        </xacro:if>
     </xacro:macro>
 </robot>

Commit message: Added multi IMU

File: xacro/gazebo.xacro (robot description, xacro)
@@ -75,5 +75,9 @@
             <visualize>true</visualize>
             <topic>__default_topic__</topic>
-            <plugin filename="libgazebo_ros_imu_sensor.so" name="imu_plugin">
+            <plugin filename="libgazebo_ros_imu_sensor.so" name="imu_plugin_trunk">
+                <ros>
+                    <namespace>/imu</namespace>
+                    <argument>~/out:=trunk_data</argument>
+                </ros>
                 <topicName>trunk_imu</topicName>
                 <bodyName>imu_link</bodyName>
@@ -83,4 +87,96 @@
                 <rpyOffset>0 0 0</rpyOffset>
                 <frameName>imu_link</frameName>
+            </plugin>
+            <pose>0 0 0 0 0 0</pose>
+        </sensor>
+    </gazebo>
+    <gazebo reference="imu_link_FL_foot">
+        <gravity>true</gravity>
+        <sensor name="imu_sensor" type="imu">
+            <always_on>true</always_on>
+            <update_rate>1000</update_rate>
+            <visualize>true</visualize>
+            <topic>__default_topic__</topic>
+            <plugin filename="libgazebo_ros_imu_sensor.so" name="imu_plugin_FL_foot">
+                <ros>
+                    <namespace>/imu</namespace>
+                    <argument>~/out:=FL_data</argument>
+                </ros>
+                <topicName>trunk_imu</topicName>
+                <bodyName>imu_link_FL_foot</bodyName>
+                <updateRateHZ>1000.0</updateRateHZ>
+                <gaussianNoise>0.0</gaussianNoise>
+                <xyzOffset>0 0 0</xyzOffset>
+                <rpyOffset>0 0 0</rpyOffset>
+                <frameName>imu_link_FL_foot</frameName>
+            </plugin>
+            <pose>0 0 0 0 0 0</pose>
+        </sensor>
+    </gazebo>
+    <gazebo reference="imu_link_FR_foot">
+        <gravity>true</gravity>
+        <sensor name="imu_sensor" type="imu">
+            <always_on>true</always_on>
+            <update_rate>1000</update_rate>
+            <visualize>true</visualize>
+            <topic>__default_topic__</topic>
+            <plugin filename="libgazebo_ros_imu_sensor.so" name="imu_plugin_FR_foot">
+                <ros>
+                    <namespace>/imu</namespace>
+                    <argument>~/out:=FR_data</argument>
+                </ros>
+                <topicName>trunk_imu</topicName>
+                <bodyName>imu_link_FR_foot</bodyName>
+                <updateRateHZ>1000.0</updateRateHZ>
+                <gaussianNoise>0.0</gaussianNoise>
+                <xyzOffset>0 0 0</xyzOffset>
+                <rpyOffset>0 0 0</rpyOffset>
+                <frameName>imu_link_FR_foot</frameName>
+            </plugin>
+            <pose>0 0 0 0 0 0</pose>
+        </sensor>
+    </gazebo>
+    <gazebo reference="imu_link_RL_foot">
+        <gravity>true</gravity>
+        <sensor name="imu_sensor" type="imu">
+            <always_on>true</always_on>
+            <update_rate>1000</update_rate>
+            <visualize>true</visualize>
+            <topic>__default_topic__</topic>
+            <plugin filename="libgazebo_ros_imu_sensor.so" name="imu_plugin_RL_foot">
+                <ros>
+                    <namespace>/imu</namespace>
+                    <argument>~/out:=RL_data</argument>
+                </ros>
+                <topicName>trunk_imu</topicName>
+                <bodyName>imu_link_RL_foot</bodyName>
+                <updateRateHZ>1000.0</updateRateHZ>
+                <gaussianNoise>0.0</gaussianNoise>
+                <xyzOffset>0 0 0</xyzOffset>
+                <rpyOffset>0 0 0</rpyOffset>
+                <frameName>imu_link_RL_foot</frameName>
+            </plugin>
+            <pose>0 0 0 0 0 0</pose>
+        </sensor>
+    </gazebo>
+    <gazebo reference="imu_link_RR_foot">
+        <gravity>true</gravity>
+        <sensor name="imu_sensor" type="imu">
+            <always_on>true</always_on>
+            <update_rate>1000</update_rate>
+            <visualize>true</visualize>
+            <topic>__default_topic__</topic>
+            <plugin filename="libgazebo_ros_imu_sensor.so" name="imu_plugin_RR_foot">
+                <ros>
+                    <namespace>/imu</namespace>
+                    <argument>~/out:=RR_data</argument>
+                </ros>
+                <topicName>trunk_imu</topicName>
+                <bodyName>imu_link_RR_foot</bodyName>
+                <updateRateHZ>1000.0</updateRateHZ>
+                <gaussianNoise>0.0</gaussianNoise>
+                <xyzOffset>0 0 0</xyzOffset>
+                <rpyOffset>0 0 0</rpyOffset>
+                <frameName>imu_link_RR_foot</frameName>
             </plugin>
             <pose>0 0 0 0 0 0</pose>

File: xacro/robot.xacro (robot description, xacro)
@@ -87,4 +87,104 @@
     <xacro:leg name="RR" mirror="-1" mirror_dae="False"  front_hind="-1" front_hind_dae="False" />
     <xacro:leg name="RL" mirror="1"  mirror_dae="True"   front_hind="-1" front_hind_dae="False" />
+    <joint name="imu_joint_FL_foot" type="fixed">
+        <parent link="FL_foot"/>
+        <child link="imu_link_FL_foot"/>
+        <origin rpy="0 0 0" xyz="0 0 0"/>
+    </joint>
+    <link name="imu_link_FL_foot">
+        <inertial>
+            <mass value="0.001"/>
+            <origin rpy="0 0 0" xyz="0 0 0"/>
+            <inertia ixx="0.0001" ixy="0" ixz="0" iyy="0.0001" iyz="0" izz="0.0001"/>
+        </inertial>
+        <visual>
+            <origin rpy="0 0 0" xyz="0 0 0"/>
+            <geometry>
+                <box size="0.001 0.001 0.001"/>
+            </geometry>
+            <!-- <material name="red"/> -->
+        </visual>
+        <collision>
+            <origin rpy="0 0 0" xyz="0 0 0"/>
+            <geometry>
+                <box size=".001 .001 .001"/>
+            </geometry>
+        </collision>
+    </link>
+    <joint name="imu_joint_FR_foot" type="fixed">
+        <parent link="FR_foot"/>
+        <child link="imu_link_FR_foot"/>
+        <origin rpy="0 0 0" xyz="0 0 0"/>
+    </joint>
+    <link name="imu_link_FR_foot">
+        <inertial>
+            <mass value="0.001"/>
+            <origin rpy="0 0 0" xyz="0 0 0"/>
+            <inertia ixx="0.0001" ixy="0" ixz="0" iyy="0.0001" iyz="0" izz="0.0001"/>
+        </inertial>
+        <visual>
+            <origin rpy="0 0 0" xyz="0 0 0"/>
+            <geometry>
+                <box size="0.001 0.001 0.001"/>
+            </geometry>
+            <!-- <material name="red"/> -->
+        </visual>
+        <collision>
+            <origin rpy="0 0 0" xyz="0 0 0"/>
+            <geometry>
+                <box size=".001 .001 .001"/>
+            </geometry>
+        </collision>
+    </link>
+    <joint name="imu_joint_RL_foot" type="fixed">
+        <parent link="RL_foot"/>
+        <child link="imu_link_RL_foot"/>
+        <origin rpy="0 0 0" xyz="0 0 0"/>
+    </joint>
+    <link name="imu_link_RL_foot">
+        <inertial>
+            <mass value="0.001"/>
+            <origin rpy="0 0 0" xyz="0 0 0"/>
+            <inertia ixx="0.0001" ixy="0" ixz="0" iyy="0.0001" iyz="0" izz="0.0001"/>
+        </inertial>
+        <visual>
+            <origin rpy="0 0 0" xyz="0 0 0"/>
+            <geometry>
+                <box size="0.001 0.001 0.001"/>
+            </geometry>
+            <!-- <material name="red"/> -->
+        </visual>
+        <collision>
+            <origin rpy="0 0 0" xyz="0 0 0"/>
+            <geometry>
+                <box size=".001 .001 .001"/>
+            </geometry>
+        </collision>
+    </link>
+    <joint name="imu_joint_RR_foot" type="fixed">
+        <parent link="RR_foot"/>
+        <child link="imu_link_RR_foot"/>
+        <origin rpy="0 0 0" xyz="0 0 0"/>
+    </joint>
+    <link name="imu_link_RR_foot">
+        <inertial>
+            <mass value="0.001"/>
+            <origin rpy="0 0 0" xyz="0 0 0"/>
+            <inertia ixx="0.0001" ixy="0" ixz="0" iyy="0.0001" iyz="0" izz="0.0001"/>
+        </inertial>
+        <visual>
+            <origin rpy="0 0 0" xyz="0 0 0"/>
+            <geometry>
+                <box size="0.001 0.001 0.001"/>
+            </geometry>
+            <!-- <material name="red"/> -->
+        </visual>
+        <collision>
+            <origin rpy="0 0 0" xyz="0 0 0"/>
+            <geometry>
+                <box size=".001 .001 .001"/>
+            </geometry>
+        </collision>
+    </link>
     <xacro:depthCamera camID="1" name="face">
         <origin rpy="${PI} 0 0" xyz="0.2785 0.0125 0.0167"/>
