Commit message: Minor

File: xacro/gazebo.xacro (robot description, xacro)
@@ -17,4 +17,10 @@
         </xacro:if>
     </gazebo>
+    <gazebo>
+        <plugin name="joint_state_publisher" filename="libgazebo_ros_joint_state_publisher.so">
+            <robotNamespace>/</robotNamespace>
+            <updateRate>250</updateRate> <!-- Match this to your simulation or controller publish rate -->
+        </plugin>
+    </gazebo>
     <!-- Show the trajectory of trunk center. -->
     <gazebo>
@@ -36,8 +42,8 @@
               <body_name>base</body_name>
               <frame_name>world</frame_name>
-              <update_rate>10.0</update_rate>
+              <update_rate>200.0</update_rate>
               <xyz_offset>0 0 0</xyz_offset>
               <rpy_offset>0 0 0</rpy_offset>
-              <gaussian_noise>0.01</gaussian_noise>
+              <gaussian_noise>0.0</gaussian_noise>
           </plugin>
         </xacro:if>
@@ -72,5 +78,5 @@
         <sensor name="imu_sensor" type="imu">
             <always_on>true</always_on>
-            <update_rate>1000</update_rate>
+            <update_rate>200</update_rate>
             <visualize>true</visualize>
             <topic>__default_topic__</topic>
@@ -82,5 +88,5 @@
                 <topicName>trunk_imu</topicName>
                 <bodyName>imu_link</bodyName>
-                <updateRateHZ>1000.0</updateRateHZ>
+                <updateRateHZ>200.0</updateRateHZ>
                 <gaussianNoise>0.0</gaussianNoise>
                 <xyzOffset>0 0 0</xyzOffset>
@@ -95,5 +101,5 @@
         <sensor name="imu_sensor" type="imu">
             <always_on>true</always_on>
-            <update_rate>1000</update_rate>
+            <update_rate>200</update_rate>
             <visualize>true</visualize>
             <topic>__default_topic__</topic>
@@ -105,5 +111,5 @@
                 <topicName>trunk_imu</topicName>
                 <bodyName>imu_link_FL_foot</bodyName>
-                <updateRateHZ>1000.0</updateRateHZ>
+                <updateRateHZ>200.0</updateRateHZ>
                 <gaussianNoise>0.0</gaussianNoise>
                 <xyzOffset>0 0 0</xyzOffset>
@@ -118,5 +124,5 @@
         <sensor name="imu_sensor" type="imu">
             <always_on>true</always_on>
-            <update_rate>1000</update_rate>
+            <update_rate>200</update_rate>
             <visualize>true</visualize>
             <topic>__default_topic__</topic>
@@ -128,5 +134,5 @@
                 <topicName>trunk_imu</topicName>
                 <bodyName>imu_link_FR_foot</bodyName>
-                <updateRateHZ>1000.0</updateRateHZ>
+                <updateRateHZ>200.0</updateRateHZ>
                 <gaussianNoise>0.0</gaussianNoise>
                 <xyzOffset>0 0 0</xyzOffset>
@@ -141,5 +147,5 @@
         <sensor name="imu_sensor" type="imu">
             <always_on>true</always_on>
-            <update_rate>1000</update_rate>
+            <update_rate>200</update_rate>
             <visualize>true</visualize>
             <topic>__default_topic__</topic>
@@ -151,5 +157,5 @@
                 <topicName>trunk_imu</topicName>
                 <bodyName>imu_link_RL_foot</bodyName>
-                <updateRateHZ>1000.0</updateRateHZ>
+                <updateRateHZ>200.0</updateRateHZ>
                 <gaussianNoise>0.0</gaussianNoise>
                 <xyzOffset>0 0 0</xyzOffset>
@@ -164,5 +170,5 @@
         <sensor name="imu_sensor" type="imu">
             <always_on>true</always_on>
-            <update_rate>1000</update_rate>
+            <update_rate>200</update_rate>
             <visualize>true</visualize>
             <topic>__default_topic__</topic>
@@ -174,5 +180,5 @@
                 <topicName>trunk_imu</topicName>
                 <bodyName>imu_link_RR_foot</bodyName>
-                <updateRateHZ>1000.0</updateRateHZ>
+                <updateRateHZ>200.0</updateRateHZ>
                 <gaussianNoise>0.0</gaussianNoise>
                 <xyzOffset>0 0 0</xyzOffset>

File: xacro/robot.xacro (robot description, xacro)
@@ -61,5 +61,5 @@
         <parent link="trunk"/>
         <child link="imu_link"/>
-        <origin rpy="0 0 0" xyz="-0.01592 -0.06659 -0.00617"/>
+        <origin rpy="0 0 0" xyz="0 0 0"/>
     </joint>
     <link name="imu_link">
