Commit message: [dev] fix LiDAR position and orientation

File: xacro/sensors.xacro (robot description, xacro)
@@ -12,5 +12,5 @@
             <parent link="trunk"/>
             <child link="lidar_mount"/>
-            <origin xyz="0.16 0 0.11" rpy="0 0 0"/>
+            <origin xyz="0.06 0 0.081" rpy="0 0 0"/>
         </joint>
         <link name="lidar_mount">
@@ -43,5 +43,5 @@
                 <parent link="lidar"/>
                 <child link="rslidar"/>
-                <origin xyz="0 0 0" rpy="0 0 1.57"/>
+                <origin xyz="0 0 0" rpy="0 0 0"/>
         </joint>
     </xacro:if>

Commit message: [minor] update lidar position

File: xacro/sensors.xacro (robot description, xacro)
@@ -12,5 +12,5 @@
             <parent link="trunk"/>
             <child link="lidar_mount"/>
-            <origin xyz="0.06 0 0.081" rpy="0 0 0"/>
+            <origin xyz="0.02 0 0.081" rpy="0 0 0"/>
         </joint>
         <link name="lidar_mount">
