Commit message: Minor

File: xacro/robot.xacro (robot description, xacro)
@@ -7,6 +7,6 @@
     <!-- <xacro:include filename="$(find go1_description)/xacro/stairs.xacro"/> -->
     <xacro:include filename="$(find go1_description)/xacro/gazebo.xacro"/>
-    <!-- <xacro:include filename="$(find go1_description)/xacro/depthCamera.xacro"/>
-    <xacro:include filename="$(find go1_description)/xacro/ultraSound.xacro"/> -->
+    <xacro:include filename="$(find go1_description)/xacro/depthCamera.xacro"/>
+    <xacro:include filename="$(find go1_description)/xacro/ultraSound.xacro"/>
     <!-- <xacro:include filename="$(find go1_gazebo)/launch/stairs.urdf.xacro"/> -->
     <!-- <xacro:stairs stairs="15" xpos="0" ypos="0" zpos="0" /> -->
@@ -87,5 +87,5 @@
     <xacro:leg name="RR" mirror="-1" mirror_dae="False"  front_hind="-1" front_hind_dae="False" />
     <xacro:leg name="RL" mirror="1"  mirror_dae="True"   front_hind="-1" front_hind_dae="False" />
-    <!-- <xacro:depthCamera camID="1" name="face">
+    <xacro:depthCamera camID="1" name="face">
         <origin rpy="${PI} 0 0" xyz="0.2785 0.0125 0.0167"/>
     </xacro:depthCamera>
@@ -124,4 +124,4 @@
     <xacro:ultraSound name="face">
         <origin rpy="0 0 0" xyz="0.2747 0.0 -0.0088"/>
-    </xacro:ultraSound> -->
+    </xacro:ultraSound>
 </robot>

File: xacro/ultraSound.xacro (robot description, xacro)
@@ -17,5 +17,5 @@
             <origin xyz="0 0 0" rpy="0 0 0"/>
             <geometry>
-                <mesh filename="package://go1_description/meshes/ultraSound.dae" scale="1 1 1"/>
+                <mesh filename="file://$(find go1_description)/meshes/ultraSound.dae" scale="1 1 1"/>
             </geometry>
             <material name="black"/>

Commit message: [add] add LiDAR sensor (velodyne)

File: xacro/robot.xacro (robot description, xacro)
@@ -125,3 +125,11 @@
         <origin rpy="0 0 0" xyz="0.2747 0.0 -0.0088"/>
     </xacro:ultraSound>
+    <!-- Sensors loading -->
+    <xacro:arg name="SENSORS" default="false"/>
+    <xacro:arg name="LIDAR" default="false"/>
+    <xacro:property name="LIDAR" value="$(arg LIDAR)"/>
+    <xacro:if value="$(arg SENSORS)">
+        <xacro:property name="LIDAR" value="true"/>
+    </xacro:if>
+    <xacro:include filename="$(find go1_description)/xacro/sensors.xacro"/>
 </robot>

Commit message: [dev] move cameras and ultrasonic sensors into sensors.xacro

File: xacro/robot.xacro (robot description, xacro)
@@ -7,6 +7,4 @@
     <!-- <xacro:include filename="$(find go1_description)/xacro/stairs.xacro"/> -->
     <xacro:include filename="$(find go1_description)/xacro/gazebo.xacro"/>
-    <xacro:include filename="$(find go1_description)/xacro/depthCamera.xacro"/>
-    <xacro:include filename="$(find go1_description)/xacro/ultraSound.xacro"/>
     <!-- <xacro:include filename="$(find go1_gazebo)/launch/stairs.urdf.xacro"/> -->
     <!-- <xacro:stairs stairs="15" xpos="0" ypos="0" zpos="0" /> -->
@@ -87,48 +85,16 @@
     <xacro:leg name="RR" mirror="-1" mirror_dae="False"  front_hind="-1" front_hind_dae="False" />
     <xacro:leg name="RL" mirror="1"  mirror_dae="True"   front_hind="-1" front_hind_dae="False" />
-    <xacro:depthCamera camID="1" name="face">
-        <origin rpy="${PI} 0 0" xyz="0.2785 0.0125 0.0167"/>
-    </xacro:depthCamera>
-    <xacro:depthCamera camID="2" name="chin">
-        <origin rpy="${PI} ${PI/2} 0" xyz="0.2522 0.0125 -0.0436"/>
-    </xacro:depthCamera>
-    <xacro:depthCamera camID="3" name="left">
-        <origin rpy="${PI} 0.2618 ${PI/2}" xyz="-0.066 0.082 -0.0176"/>
-    </xacro:depthCamera>
-    <xacro:depthCamera camID="4" name="right">
-        <origin rpy="${PI} 0.2618 ${-PI/2}" xyz="-0.041 -0.082 -0.0176"/>
-    </xacro:depthCamera>
-    <xacro:depthCamera camID="5" name="rearDown">
-        <origin rpy="${PI} ${PI/2} 0" xyz="-0.0825 0.0125 -0.04365"/>
-    </xacro:depthCamera>
-    <joint name="camera_laserscan_joint_left" type="fixed">
-        <origin rpy="0 0.2618 0" xyz="0 0 0"/>
-        <parent link="camera_left"/>
-        <child link="camera_laserscan_link_left"/>
-    </joint>
-    <link name="camera_laserscan_link_left">
-    </link>
-    <joint name="camera_laserscan_joint_right" type="fixed">
-        <origin rpy="0 0.2618 0" xyz="0 0 0"/>
-        <parent link="camera_right"/>
-        <child link="camera_laserscan_link_right"/>
-    </joint>
-    <link name="camera_laserscan_link_right">
-    </link>
-    <xacro:ultraSound name="left">
-        <origin rpy="0 0.2618 ${PI/2}" xyz="-0.0535  0.0826 0.00868"/>
-    </xacro:ultraSound>
-    <xacro:ultraSound name="right">
-        <origin rpy="0 0.2618 ${-PI/2}" xyz="-0.0535 -0.0826 0.00868"/>
-    </xacro:ultraSound>
-    <xacro:ultraSound name="face">
-        <origin rpy="0 0 0" xyz="0.2747 0.0 -0.0088"/>
-    </xacro:ultraSound>
     <!-- Sensors loading -->
     <xacro:arg name="SENSORS" default="false"/>
     <xacro:arg name="LIDAR" default="false"/>
+    <xacro:arg name="CAMERAS" default="false"/>
+    <xacro:arg name="ULTRASONIC" default="false"/>
     <xacro:property name="LIDAR" value="$(arg LIDAR)"/>
+    <xacro:property name="CAMERAS" value="$(arg CAMERAS)"/>
+    <xacro:property name="ULTRASONIC" value="$(arg ULTRASONIC)"/>
     <xacro:if value="$(arg SENSORS)">
         <xacro:property name="LIDAR" value="true"/>
+        <xacro:property name="CAMERAS" value="true"/>
+        <xacro:property name="ULTRASONIC" value="true"/>
     </xacro:if>
     <xacro:include filename="$(find go1_description)/xacro/sensors.xacro"/>

File: xacro/sensors.xacro (robot description, xacro)
@@ -2,5 +2,6 @@
 <robot xmlns:xacro="http://www.ros.org/wiki/xacro">
     <xacro:include filename="$(find sensors_description)/xacro/VLP-16.urdf.xacro"/>
-    <xacro:include filename="$(find sensors_description)/xacro/realsense_d430.urdf.xacro" />
+    <xacro:include filename="$(find go1_description)/xacro/depthCamera.xacro"/>
+    <xacro:include filename="$(find go1_description)/xacro/ultraSound.xacro"/>
     <!-- Lidar -->
     <xacro:if value="${LIDAR}">
@@ -45,3 +46,55 @@
         </joint>
     </xacro:if>
+    <!-- Cameras -->
+    <xacro:if value="${CAMERAS}">
+        <!-- Face -->
+        <xacro:depthCamera camID="1" name="face">
+            <origin rpy="${PI} 0 0" xyz="0.2785 0.0125 0.0167"/>
+        </xacro:depthCamera>
+        <!-- Chin -->
+        <xacro:depthCamera camID="2" name="chin">
+            <origin rpy="${PI} ${PI/2} 0" xyz="0.2522 0.0125 -0.0436"/>
+        </xacro:depthCamera>
+        <!-- Left -->
+        <xacro:depthCamera camID="3" name="left">
+            <origin rpy="${PI} 0.2618 ${PI/2}" xyz="-0.066 0.082 -0.0176"/>
+        </xacro:depthCamera>
+        <!-- Right -->
+        <xacro:depthCamera camID="4" name="right">
+            <origin rpy="${PI} 0.2618 ${-PI/2}" xyz="-0.041 -0.082 -0.0176"/>
+        </xacro:depthCamera>
+        <!-- Rear Down -->
+        <xacro:depthCamera camID="5" name="rearDown">
+            <origin rpy="${PI} ${PI/2} 0" xyz="-0.0825 0.0125 -0.04365"/>
+        </xacro:depthCamera>
+        <joint name="camera_laserscan_joint_left" type="fixed">
+            <origin rpy="0 0.2618 0" xyz="0 0 0"/>
+            <parent link="camera_left"/>
+            <child link="camera_laserscan_link_left"/>
+        </joint>
+        <link name="camera_laserscan_link_left">
+        </link>
+        <joint name="camera_laserscan_joint_right" type="fixed">
+            <origin rpy="0 0.2618 0" xyz="0 0 0"/>
+            <parent link="camera_right"/>
+            <child link="camera_laserscan_link_right"/>
+        </joint>
+        <link name="camera_laserscan_link_right">
+        </link>
+    </xacro:if>
+    <!-- Ultrasonic Sensors -->
+    <xacro:if value="${ULTRASONIC}">
+        <!--Left-->
+        <xacro:ultraSound name="left">
+            <origin rpy="0 0.2618 ${PI/2}" xyz="-0.0535  0.0826 0.00868"/>
+        </xacro:ultraSound>
+        <!--Right-->
+        <xacro:ultraSound name="right">
+            <origin rpy="0 0.2618 ${-PI/2}" xyz="-0.0535 -0.0826 0.00868"/>
+        </xacro:ultraSound>
+        <!--Face-->
+        <xacro:ultraSound name="face">
+            <origin rpy="0 0 0" xyz="0.2747 0.0 -0.0088"/>
+        </xacro:ultraSound>
+    </xacro:if>
 </robot>

Commit message: [minor] minor changes

File: xacro/robot.xacro (robot description, xacro)
@@ -1,12 +1,9 @@
 <?xml version="1.0"?>
-<robot name="go1" xmlns:xacro="http://www.ros.org/wiki/xacro">
+<robot name="go1_description" xmlns:xacro="http://www.ros.org/wiki/xacro">
     <xacro:arg name="DEBUG" default="false"/>
     <xacro:include filename="$(find go1_description)/xacro/const.xacro"/>
     <xacro:include filename="$(find go1_description)/xacro/materials.xacro"/>
     <xacro:include filename="$(find go1_description)/xacro/leg.xacro"/>
-    <!-- <xacro:include filename="$(find go1_description)/xacro/stairs.xacro"/> -->
     <xacro:include filename="$(find go1_description)/xacro/gazebo.xacro"/>
-    <!-- <xacro:include filename="$(find go1_gazebo)/launch/stairs.urdf.xacro"/> -->
-    <!-- <xacro:stairs stairs="15" xpos="0" ypos="0" zpos="0" /> -->
     <!-- Rotor related joint and link is only for demonstrate location. -->
     <!-- Actually, the rotor will rotate and the joint is not fixed. Reduction ratio should be considered. -->
@@ -17,8 +14,8 @@
             <origin rpy="0 0 0" xyz="0 0 0"/>
             <parent link="world"/>
-            <child link="base"/>
+            <child link="trunk"/>
         </joint>
     </xacro:if>
-    <link name="base">
+    <!-- <link name="base">
         <visual>
             <origin rpy="0 0 0" xyz="0 0 0"/>
@@ -32,5 +29,5 @@
         <parent link="base"/>
         <child link="trunk"/>
-    </joint>
+    </joint> -->
     <link name="trunk">
         <visual>
@@ -39,5 +36,5 @@
                 <mesh filename="file://$(find go1_description)/meshes/trunk.dae" scale="1 1 1"/>
             </geometry>
-            <!-- <material name="orange"/> -->
+            <material name="orange"/>
         </visual>
         <collision>
@@ -72,5 +69,5 @@
                 <box size="0.001 0.001 0.001"/>
             </geometry>
-            <!-- <material name="red"/> -->
+            <material name="red"/>
         </visual>
         <collision>

Commit message: renamed ultrasonic into ultrasound

File: xacro/robot.xacro (robot description, xacro)
@@ -89,9 +89,9 @@
     <xacro:property name="LIDAR" value="$(arg LIDAR)"/>
     <xacro:property name="CAMERAS" value="$(arg CAMERAS)"/>
-    <xacro:property name="ULTRASONIC" value="$(arg ULTRASONIC)"/>
+    <xacro:property name="ULTRASOUND" value="$(arg ULTRASONIC)"/>
     <xacro:if value="$(arg SENSORS)">
         <xacro:property name="LIDAR" value="true"/>
         <xacro:property name="CAMERAS" value="true"/>
-        <xacro:property name="ULTRASONIC" value="true"/>
+        <xacro:property name="ULTRASOUND" value="true"/>
     </xacro:if>
     <xacro:include filename="$(find go1_description)/xacro/sensors.xacro"/>
