Commit message: Added cameras and Lidar sensors

File: urdf/robot_old.urdf (robot description, URDF)
Before this commit: robot go1, 38 links, 37 joints
Links:
- removed link lidar_link
Joints:
- removed joint lidar_joint

File: urdf/robot_old_old.urdf (robot description, URDF)
Before this commit: robot go1, 38 links, 37 joints
Links:
- removed link lidar_link
Joints:
- removed joint lidar_joint

File: xacro/depthCamera.xacro (robot description, xacro)
@@ -76,4 +76,53 @@
 		<!--            </sensor>-->
 		<!--        </gazebo>-->
+		       <gazebo reference="camera_${name}">
+		           <!-- &lt;!&ndash; <material>Gazebo/Black</material> &ndash;&gt; -->
+				   <material>Gazebo/Black</material>
+		           <sensor name="camera_${name}_camera" type="depth">
+		               <update_rate>16</update_rate>
+		               <camera>
+		                   <horizontal_fov>2.094</horizontal_fov>
+		                   <image>
+		                       <width>928</width>
+		                       <height>800</height>
+		                       <format>R8G8B8</format>
+		                   </image>
+							<vertical>
+								<samples>32</samples>
+								<min_angle>-0.5353</min_angle>
+								<max_angle>0.1862</max_angle>
+							</vertical>
+		                   <clip>
+		                       <near>0.1</near>
+		                       <far>5</far>
+		                   </clip>
+		               </camera>
+		<!--                <plugin name="camera_${name}_controller" filename="libgazebo_ros_openni_kinect.so">-->
+		<!--                    <baseline>0.025</baseline>-->
+		<!--                    <alwaysOn>true</alwaysOn>-->
+		<!--                    <updateRate>0.0</updateRate>-->
+		<!--                    <cameraName>camera_${name}_ir</cameraName>-->
+		<!--                    <imageTopicName>/camera_${name}/color/image_raw</imageTopicName>-->
+		<!--                    <cameraInfoTopicName>/camera_${name}/color/camera_info</cameraInfoTopicName>-->
+		<!--                    <depthImageTopicName>/camera_${name}/depth/image_raw</depthImageTopicName>-->
+		<!--                    <depthImageInfoTopicName>/camera_${name}/depth/camera_info</depthImageInfoTopicName>-->
+		<!--                    &lt;!&ndash; <pointCloudTopicName>/camera_${name}/depth/points</pointCloudTopicName> &ndash;&gt;-->
+		<!--                    <pointCloudTopicName>/cam${camID}/point_cloud_${name}</pointCloudTopicName>-->
+		<!--                    <frameName>camera_optical_${name}</frameName>-->
+		<!--                    <pointCloudCutoff>0.1</pointCloudCutoff>-->
+		<!--                    <pointCloudCutoffMax>1.5</pointCloudCutoffMax>-->
+		<!--                    <distortionK1>0.0</distortionK1>-->
+		<!--                    <distortionK2>0.0</distortionK2>-->
+		<!--                    <distortionK3>0.0</distortionK3>-->
+		<!--                    <distortionT1>0.0</distortionT1>-->
+		<!--                    <distortionT2>0.0</distortionT2>-->
+		<!--                    <CxPrime>0</CxPrime>-->
+		<!--                    <Cx>0.0045</Cx>-->
+		<!--                    <Cy>0.0039</Cy>-->
+		<!--                    <focalLength>0</focalLength>-->
+		<!--                    <hackBaseline>0</hackBaseline>-->
+		<!--                </plugin>-->
+		           </sensor>
+		       </gazebo>
 	</xacro:macro>
 </robot>

File: xacro/gazebo.xacro (robot description, xacro)
@@ -309,3 +309,45 @@
 	<xacro:ft_sensor name="RF"/>
 	<xacro:ft_sensor name="RH"/> -->
+	<gazebo reference="lidar_link">
+		<sensor name="gpu_lidar" type="gpu_lidar">
+			<update_rate>10</update_rate>
+			<topic>scan</topic>
+			<gz_frame_id>lidar_link</gz_frame_id>
+			<lidar>
+				<scan>
+					<horizontal>
+						<samples>32</samples>
+						<!--(max_angle-min_angle)/samples * resolution -->
+						<resolution>1</resolution>
+						<min_angle>-3.14156</min_angle>
+						<max_angle>3.14156</max_angle>
+					</horizontal>
+					<!-- Dirty hack for fake lidar detections with ogre 1 rendering in VM -->
+					<!-- <vertical>
+						<samples>3</samples>
+						<min_angle>-0.001</min_angle>
+						<max_angle>0.001</max_angle>
+					</vertical> -->
+					<vertical>
+						<samples>32</samples>
+						<min_angle>-0.1</min_angle>
+						<max_angle>0.1862</max_angle>
+					</vertical>
+				</scan>
+				<range>
+					<min>0.05</min>
+					<max>10.0</max>
+					<resolution>0.01</resolution>
+				</range>
+				<noise>
+					<type>gaussian</type>
+					<mean>0.0</mean>
+					<stddev>0.01</stddev>
+				</noise>
+				<frame_id>lidar_link</frame_id>
+			</lidar>
+			<always_on>1</always_on>
+			<visualize>true</visualize>
+		</sensor>
+	</gazebo>
 </robot>

File: xacro/robot.xacro (robot description, xacro)
@@ -9,4 +9,5 @@
 	<xacro:include filename="$(find go1_description)/xacro/depthCamera.xacro"/>
 	<xacro:include filename="$(find go1_description)/xacro/ultraSound.xacro"/>
+	<xacro:include filename="$(find go1_description)/xacro/lidar.xacro"/>
 	<xacro:if value="$(arg GAZEBO)">
 		<xacro:if value="$(arg CLASSIC)">
@@ -135,3 +136,6 @@
 		<origin rpy="0 0 0" xyz="0.2747 0.0 -0.0088"/>
 	</xacro:ultraSound>
+	<xacro:lidar>
+        <origin xyz="0.0 0 0.04675" rpy="0.0 0 0"/>
+	</xacro:lidar>
 </robot>
