Commit message: Working urdf version

File: urdf/robot.urdf (robot description, URDF)
Before this commit: robot go1, 37 links, 36 joints
Links:
- link LF_calf: geometry collision box size=0.213 0.016 0.016; visual mesh filename=file:///home/ocs_2/quadruped_nmpc_hierarchical_ws/install/g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 scale=1 1 1
- link LF_hip: geometry collision cylinder length=0.04 radius=0.046; visual mesh filename=file:///home/ocs_2/quadruped_nmpc_hierarchical_ws/install/g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 scale=1 1 1
- link LF_thigh: geometry collision box size=0.213 0.0245 0.034; visual mesh filename=file:///home/ocs_2/quadruped_nmpc_hierarchical_ws/install/g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 scale=1 1 1
- link LH_calf: geometry collision box size=0.213 0.016 0.016; visual mesh filename=file:///home/ocs_2/quadruped_nmpc_hierarchical_ws/install/g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 scale=1 1 1
- link LH_hip: geometry collision cylinder length=0.04 radius=0.046; visual mesh filename=file:///home/ocs_2/quadruped_nmpc_hierarchical_ws/install/g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 scale=1 1 1
- link LH_thigh: geometry collision box size=0.213 0.0245 0.034; visual mesh filename=file:///home/ocs_2/quadruped_nmpc_hierarchical_ws/install/g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 scale=1 1 1
- link RF_calf: geometry collision box size=0.213 0.016 0.016; visual mesh filename=file:///home/ocs_2/quadruped_nmpc_hierarchical_ws/install/g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 scale=1 1 1
- link RF_hip: geometry collision cylinder length=0.04 radius=0.046; visual mesh filename=file:///home/ocs_2/quadruped_nmpc_hierarchical_ws/install/g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 scale=1 1 1
- link RF_thigh: geometry collision box size=0.213 0.0245 0.034; visual mesh filename=file:///home/ocs_2/quadruped_nmpc_hierarchical_ws/install/g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 scale=1 1 1
- link RH_calf: geometry collision box size=0.213 0.016 0.016; visual mesh filename=file:///home/ocs_2/quadruped_nmpc_hierarchical_ws/install/g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 scale=1 1 1
- link RH_hip: geometry collision cylinder length=0.04 radius=0.046; visual mesh filename=file:///home/ocs_2/quadruped_nmpc_hierarchical_ws/install/g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 scale=1 1 1
- link RH_thigh: geometry collision box size=0.213 0.0245 0.034; visual mesh filename=file:///home/ocs_2/quadruped_nmpc_hierarchical_ws/install/g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 scale=1 1 1
- link base: geometry collision box size=0.3762 0.0935 0.114; visual mesh filename=file:///home/ocs_2/quadruped_nmpc_hierarchical_ws/install/g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 scale=1 1 1
- link camera_chin: geometry collision box size=.001 .001 .001; visual mesh filename=file:///home/ocs_2/quadruped_nmpc_hierarchical_ws/install/g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 scale=1 1 1
- link camera_face: geometry collision box size=.001 .001 .001; visual mesh filename=file:///home/ocs_2/quadruped_nmpc_hierarchical_ws/install/g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 scale=1 1 1
- link camera_left: geometry collision box size=.001 .001 .001; visual mesh filename=file:///home/ocs_2/quadruped_nmpc_hierarchical_ws/install/g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 scale=1 1 1
- link camera_rearDown: geometry collision box size=.001 .001 .001; visual mesh filename=file:///home/ocs_2/quadruped_nmpc_hierarchical_ws/install/g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 scale=1 1 1
- link camera_right: geometry collision box size=.001 .001 .001; visual mesh filename=file:///home/ocs_2/quadruped_nmpc_hierarchical_ws/install/g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 scale=1 1 1
- link ultraSound_face: geometry collision box size=.001 .001 .001; visual mesh filename=file:///home/ocs_2/quadruped_nmpc_hierarchical_ws/install/g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 scale=1 1 1
- link ultraSound_left: geometry collision box size=.001 .001 .001; visual mesh filename=file:///home/ocs_2/quadruped_nmpc_hierarchical_ws/install/g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 scale=1 1 1
- link ultraSound_right: geometry collision box size=.001 .001 .001; visual mesh filename=file:///home/ocs_2/quadruped_nmpc_hierarchical_ws/install/g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 scale=1 1 1

Commit message: minor

File: urdf/robot.urdf (robot description, URDF)
Before this commit: robot go1, 37 links, 36 joints
Links:
- link LF_calf: geometry collision box size=0.213 0.016 0.016; visual mesh filename=file:///home/quadruped_nmpc_hierarchical/quadruped_nmpc_hie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 scale=1 1 1
- link LF_hip: geometry collision cylinder length=0.04 radius=0.046; visual mesh filename=file:///home/quadruped_nmpc_hierarchical/quadruped_nmpc_hie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 scale=1 1 1
- link LF_thigh: geometry collision box size=0.213 0.0245 0.034; visual mesh filename=file:///home/quadruped_nmpc_hierarchical/quadruped_nmpc_hie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 scale=1 1 1
- link LH_calf: geometry collision box size=0.213 0.016 0.016; visual mesh filename=file:///home/quadruped_nmpc_hierarchical/quadruped_nmpc_hie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 scale=1 1 1
- link LH_hip: geometry collision cylinder length=0.04 radius=0.046; visual mesh filename=file:///home/quadruped_nmpc_hierarchical/quadruped_nmpc_hie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 scale=1 1 1
- link LH_thigh: geometry collision box size=0.213 0.0245 0.034; visual mesh filename=file:///home/quadruped_nmpc_hierarchical/quadruped_nmpc_hie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 scale=1 1 1
- link RF_calf: geometry collision box size=0.213 0.016 0.016; visual mesh filename=file:///home/quadruped_nmpc_hierarchical/quadruped_nmpc_hie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 scale=1 1 1
- link RF_hip: geometry collision cylinder length=0.04 radius=0.046; visual mesh filename=file:///home/quadruped_nmpc_hierarchical/quadruped_nmpc_hie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 scale=1 1 1
- link RF_thigh: geometry collision box size=0.213 0.0245 0.034; visual mesh filename=file:///home/quadruped_nmpc_hierarchical/quadruped_nmpc_hie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 scale=1 1 1
- link RH_calf: geometry collision box size=0.213 0.016 0.016; visual mesh filename=file:///home/quadruped_nmpc_hierarchical/quadruped_nmpc_hie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 scale=1 1 1
- link RH_hip: geometry collision cylinder length=0.04 radius=0.046; visual mesh filename=file:///home/quadruped_nmpc_hierarchical/quadruped_nmpc_hie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 scale=1 1 1
- link RH_thigh: geometry collision box size=0.213 0.0245 0.034; visual mesh filename=file:///home/quadruped_nmpc_hierarchical/quadruped_nmpc_hie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 scale=1 1 1
- link base: geometry collision box size=0.3762 0.0935 0.114; visual mesh filename=file:///home/quadruped_nmpc_hierarchical/quadruped_nmpc_hie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 scale=1 1 1
- link camera_chin: geometry collision box size=.001 .001 .001; visual mesh filename=file:///home/quadruped_nmpc_hierarchical/quadruped_nmpc_hie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 scale=1 1 1
- link camera_face: geometry collision box size=.001 .001 .001; visual mesh filename=file:///home/quadruped_nmpc_hierarchical/quadruped_nmpc_hie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 scale=1 1 1
- link camera_left: geometry collision box size=.001 .001 .001; visual mesh filename=file:///home/quadruped_nmpc_hierarchical/quadruped_nmpc_hie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 scale=1 1 1
- link camera_rearDown: geometry collision box size=.001 .001 .001; visual mesh filename=file:///home/quadruped_nmpc_hierarchical/quadruped_nmpc_hie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 scale=1 1 1
- link camera_right: geometry collision box size=.001 .001 .001; visual mesh filename=file:///home/quadruped_nmpc_hierarchical/quadruped_nmpc_hie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 scale=1 1 1
- link ultraSound_face: geometry collision box size=.001 .001 .001; visual mesh filename=file:///home/quadruped_nmpc_hierarchical/quadruped_nmpc_hie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 scale=1 1 1
- link ultraSound_left: geometry collision box size=.001 .001 .001; visual mesh filename=file:///home/quadruped_nmpc_hierarchical/quadruped_nmpc_hie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 scale=1 1 1
- link ultraSound_right: geometry collision box size=.001 .001 .001; visual mesh filename=file:///home/quadruped_nmpc_hierarchical/quadruped_nmpc_hie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 scale=1 1 1

Commit message: Added Lidar gps and imu sensors

File: urdf/robot.urdf (robot description, URDF)
Before this commit: robot go1, 38 links, 37 joints
Links:
- added link gps_link
Joints:
- added joint gps_joint: type fixed, parent base, child gps_link, origin xyz=0 0 0 rpy=0 0 0

File: xacro/gazebo.xacro (robot description, xacro)
@@ -323,5 +323,4 @@
 						<max_angle>3.14156</max_angle>
 					</horizontal>
-					<!-- Dirty hack for fake lidar detections with ogre 1 rendering in VM -->
 					<!-- <vertical>
 						<samples>3</samples>
@@ -351,3 +350,11 @@
 		</sensor>
 	</gazebo>
+	<gazebo reference="gps_link">
+		<sensor name="gps" type="navsat">
+			<always_on>1</always_on>
+			<update_rate>10</update_rate>
+			<topic>gps</topic>
+			<gz_frame_id>gps_link</gz_frame_id>
+		</sensor>
+	</gazebo>
 </robot>

File: xacro/lidar.xacro (robot description, xacro)
@@ -18,5 +18,5 @@
                 />
             </inertial>
-            <collision name='collision'>
+            <collision name='lidar_link_collision'>
                 <origin xyz="0 0 0" rpy="1.57 0 0"/>
                 <geometry>
@@ -24,5 +24,5 @@
                 </geometry>
             </collision>
-            <visual name='scan_link_visual'>
+            <visual name='lidar_link_visual'>
                 <origin xyz="0 0 0" rpy="1.57 0 0"/>
                 <geometry>

File: xacro/robot.xacro (robot description, xacro)
@@ -10,4 +10,5 @@
 	<xacro:include filename="$(find go1_description)/xacro/ultraSound.xacro"/>
 	<xacro:include filename="$(find go1_description)/xacro/lidar.xacro"/>
+	<xacro:include filename="$(find sensors_description)/xacro/gps.xacro"/>
 	<xacro:if value="$(arg GAZEBO)">
 		<xacro:if value="$(arg CLASSIC)">
@@ -139,3 +140,6 @@
         <origin xyz="0.0 0 0.04675" rpy="0.0 0 0"/>
 	</xacro:lidar>
+	<xacro:gps parent="base">
+		<origin xyz="0.0 0.0 0.0" rpy="0.0 0.0 0.0"/>
+	</xacro:gps>
 </robot>

Commit message: gz harmonic working version

File: urdf/robot.urdf (robot description, URDF)
Before this commit: robot go1, 39 links, 38 joints
Links:
- removed link lidar_link
- added link lidar, mass 0.01
- added link lidar_base_link, mass 0.87; collision cylinder length=0.12 radius=0.055; visual mesh filename=file:///home/quadruped_nmpc_hierarchical/quadruped_nmpc_hie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 scale=0.001 0.001 0.001
Joints:
- removed joint lidar_joint
- added joint lidar_base_mount_joint: type fixed, parent base, child lidar_base_link, origin xyz=0 0 0.04675 rpy=0 0 0
- added joint lidar_base_scan_joint: type fixed, parent lidar_base_link, child lidar, origin xyz=0 0 0.039 rpy=0 0 0

File: urdf/robot_old.urdf (robot description, URDF)
Before this commit: robot go1, 37 links, 36 joints
Links:
- added link gps_link
- added link lidar_link, mass 1e-5; collision mesh filename=file:///home/quadruped_nmpc_hierarchical/quadruped_nmpc_hie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 scale=0.001 0.001 0.001; visual mesh filename=file:///home/quadruped_nmpc_hierarchical/quadruped_nmpc_hie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 scale=0.001 0.001 0.001
Joints:
- added joint gps_joint: type fixed, parent base, child gps_link, origin xyz=0 0 0 rpy=0 0 0
- added joint lidar_joint: type fixed, parent base, child lidar_link, origin xyz=0.0 0 0.04675 rpy=0.0 0 0, axis 0 0 1

File: xacro/gazebo.xacro (robot description, xacro)
@@ -305,9 +305,5 @@
 		</sensor>
 	</gazebo>
-	<!-- <xacro:ft_sensor name="LF"/>
-	<xacro:ft_sensor name="LH"/>
-	<xacro:ft_sensor name="RF"/>
-	<xacro:ft_sensor name="RH"/> -->
-	<gazebo reference="lidar_link">
+	<!-- <gazebo reference="lidar_link">
 		<sensor name="gpu_lidar" type="gpu_lidar">
 			<update_rate>10</update_rate>
@@ -317,15 +313,9 @@
 				<scan>
 					<horizontal>
-						<samples>32</samples>
-						<!--(max_angle-min_angle)/samples * resolution -->
+						<samples>900</samples>
 						<resolution>1</resolution>
 						<min_angle>-3.14156</min_angle>
 						<max_angle>3.14156</max_angle>
 					</horizontal>
-					<!-- <vertical>
-						<samples>3</samples>
-						<min_angle>-0.001</min_angle>
-						<max_angle>0.001</max_angle>
-					</vertical> -->
 					<vertical>
 						<samples>32</samples>
@@ -342,5 +332,5 @@
 					<type>gaussian</type>
 					<mean>0.0</mean>
-					<stddev>0.01</stddev>
+					<stddev>0.008</stddev>
 				</noise>
 				<frame_id>lidar_link</frame_id>
@@ -349,5 +339,5 @@
 			<visualize>true</visualize>
 		</sensor>
-	</gazebo>
+	</gazebo> -->
 	<gazebo reference="gps_link">
 		<sensor name="gps" type="navsat">

File: xacro/robot.xacro (robot description, xacro)
@@ -9,6 +9,8 @@
 	<xacro:include filename="$(find go1_description)/xacro/depthCamera.xacro"/>
 	<xacro:include filename="$(find go1_description)/xacro/ultraSound.xacro"/>
-	<xacro:include filename="$(find go1_description)/xacro/lidar.xacro"/>
+	<!-- <xacro:include filename="$(find go1_description)/xacro/lidar.xacro"/> -->
 	<xacro:include filename="$(find sensors_description)/xacro/gps.xacro"/>
+	<xacro:include filename="$(find sensors_description)/xacro/robosense_lidar_16.xacro"/>
+	<xacro:include filename="$(find sensors_description)/xacro/lidar_3d.gazebo.xacro"/>
 	<xacro:if value="$(arg GAZEBO)">
 		<xacro:if value="$(arg CLASSIC)">
@@ -137,7 +139,14 @@
 		<origin rpy="0 0 0" xyz="0.2747 0.0 -0.0088"/>
 	</xacro:ultraSound>
-	<xacro:lidar>
+	<!-- <xacro:lidar>
         <origin xyz="0.0 0 0.04675" rpy="0.0 0 0"/>
-	</xacro:lidar>
+	</xacro:lidar> -->
+	<xacro:robosense_lidar_16
+		name="lidar"
+		parent="base"
+		sim_ignition="true"
+		topic="/lidar_3d">
+		<origin xyz="0 0 0.04675" rpy="0 0 0"/>
+	</xacro:robosense_lidar_16>
 	<xacro:gps parent="base">
 		<origin xyz="0.0 0.0 0.0" rpy="0.0 0.0 0.0"/>

Commit message: lidar to rslidar

File: urdf/robot.urdf (robot description, URDF)
Before this commit: robot go1, 40 links, 39 joints
Links:
- removed link lidar
- removed link lidar_base_link
- added link rslidar, mass 0.01
- added link rslidar_base_link, mass 0.87; collision cylinder length=0.12 radius=0.055; visual mesh filename=file:///home/quadruped_nmpc_hierarchical/quadruped_nmpc_hie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 scale=0.001 0.001 0.001
Joints:
- removed joint lidar_base_mount_joint
- removed joint lidar_base_scan_joint
- added joint rslidar_base_mount_joint: type fixed, parent base, child rslidar_base_link, origin xyz=0 0 0.04675 rpy=0 0 0
- added joint rslidar_base_scan_joint: type fixed, parent rslidar_base_link, child rslidar, origin xyz=0 0 0.039 rpy=0 0 0

File: xacro/robot.xacro (robot description, xacro)
@@ -143,5 +143,5 @@
 	</xacro:lidar> -->
 	<xacro:robosense_lidar_16
-		name="lidar"
+		name="rslidar"
 		parent="base"
 		sim_ignition="true"
