Commit message: Minor

File: go1_description/xacro/gazebo.xacro (robot description, xacro)
@@ -2,350 +2,352 @@
 <robot xmlns:xacro="http://www.ros.org/wiki/xacro">
 	<xacro:include filename="$(find go1_description)/xacro/ft_sensor.xacro"/>
-	<ros2_control name="GazeboSystem" type="system">
-		<hardware>
-			<plugin>gz_ros2_control/GazeboSimSystem</plugin>
-		</hardware>
-		<!-- <hardware>
-			<plugin>ign_ros2_control/IgnitionSystem</plugin>
-		</hardware> -->
-		<joint name="LF_HAA">
-			<command_interface name="effort"/>
-			<command_interface name="velocity" initial_value="0.0"/>
-			<state_interface name="position">
-				<param name="initial_value">0.0</param>
-			</state_interface>
-			<state_interface name="velocity"/>
-			<state_interface name="effort"/>
-		</joint>
-		<joint name="LF_HFE">
-			<command_interface name="effort"/>
-			<command_interface name="velocity" initial_value="0.0"/>
-			<state_interface name="position">
-				<param name="initial_value">0.72</param>
-			</state_interface>
-			<state_interface name="velocity"/>
-			<state_interface name="effort"/>
-		</joint>
-		<joint name="LF_KFE">
-			<command_interface name="effort"/>
-			<command_interface name="velocity" initial_value="0.0"/>
-			<state_interface name="position">
-				<param name="initial_value">-1.44</param>
-			</state_interface>
-			<state_interface name="velocity"/>
-			<state_interface name="effort"/>
-		</joint>
-		<joint name="LH_HAA">
-			<command_interface name="effort"/>
-			<command_interface name="velocity" initial_value="0.0"/>
-						<state_interface name="position">
-				<param name="initial_value">0.0</param>
-			</state_interface>
-			<state_interface name="velocity"/>
-			<state_interface name="effort"/>
-		</joint>
-		<joint name="LH_HFE">
-			<command_interface name="effort"/>
-			<command_interface name="velocity" initial_value="0.0"/>
-			<state_interface name="position">
-				<param name="initial_value">0.72</param>
-			</state_interface>
-			<state_interface name="velocity"/>
-			<state_interface name="effort"/>
-		</joint>
-		<joint name="LH_KFE">
-			<command_interface name="effort"/>
-			<command_interface name="velocity" initial_value="0.0"/>
-			<state_interface name="position">
-				<param name="initial_value">-1.44</param>
-			</state_interface>
-			<state_interface name="velocity"/>
-			<state_interface name="effort"/>
-		</joint>
-		<joint name="RF_HAA">
-			<command_interface name="effort"/>
-			<command_interface name="velocity" initial_value="0.0"/>
-			<state_interface name="position">
-				<param name="initial_value">0.0</param>
-			</state_interface>
-			<state_interface name="velocity"/>
-			<state_interface name="effort"/>
-		</joint>
-		<joint name="RF_HFE">
-			<command_interface name="effort"/>
-			<command_interface name="velocity" initial_value="0.0"/>
-			<state_interface name="position">
-				<param name="initial_value">0.72</param>
-			</state_interface>
-			<state_interface name="velocity"/>
-			<state_interface name="effort"/>
-		</joint>
-		<joint name="RF_KFE">
-			<command_interface name="effort"/>
-			<command_interface name="velocity" initial_value="0.0"/>
-			<state_interface name="position">
-				<param name="initial_value">-1.44</param>
-			</state_interface>
-			<state_interface name="velocity"/>
-			<state_interface name="effort"/>
-		</joint>
-		<joint name="RH_HAA">
-			<command_interface name="effort"/>
-			<command_interface name="velocity" initial_value="0.0"/>
-			<state_interface name="position">
-				<param name="initial_value">0.0</param>
-			</state_interface>
-			<state_interface name="velocity"/>
-			<state_interface name="effort"/>
-		</joint>
-		<joint name="RH_HFE">
-			<command_interface name="effort"/>
-			<command_interface name="velocity" initial_value="0.0"/>
-			<state_interface name="position">
-				<param name="initial_value">0.72</param>
-			</state_interface>
-			<state_interface name="velocity"/>
-			<state_interface name="effort"/>
-		</joint>
-		<joint name="RH_KFE">
-			<command_interface name="effort"/>
-			<command_interface name="velocity" initial_value="0.0"/>
-			<state_interface name="position">
-				<param name="initial_value">-1.44</param>
-			</state_interface>
-			<state_interface name="velocity"/>
-			<state_interface name="effort"/>
-		</joint>
-		<sensor name="imu_sensor">
-			<state_interface name="orientation.x"/>
-			<state_interface name="orientation.y"/>
-			<state_interface name="orientation.z"/>
-			<state_interface name="orientation.w"/>
-			<state_interface name="angular_velocity.x"/>
-			<state_interface name="angular_velocity.y"/>
-			<state_interface name="angular_velocity.z"/>
-			<state_interface name="linear_acceleration.x"/>
-			<state_interface name="linear_acceleration.y"/>
-			<state_interface name="linear_acceleration.z"/>
-		</sensor>
-	</ros2_control>
-	<gazebo>
-		<plugin filename="gz_ros2_control-system" name="gz_ros2_control::GazeboSimROS2ControlPlugin">
-			<parameters>$(find go1_description)/config/gazebo.yaml</parameters>
-		</plugin>
-		<plugin filename="gz-sim-imu-system"
-						name="gz::sim::systems::Imu">
-		</plugin>
-	</gazebo>
-	<gazebo reference="base">
-		<mu1>0.6</mu1>
-		<mu2>0.6</mu2>
-		<self_collide>1</self_collide>
-	</gazebo>
-	<gazebo>
-		<plugin name="gz::sim::systems::OdometryPublisher" filename="gz-sim-odometry-publisher-system">
-			<robot_base_frame>/go1/base</robot_base_frame>
-			<dimensions>3</dimensions>
-		</plugin>
-	</gazebo>
-	<gazebo reference="imu_link">
-		<sensor name="imu_sensor" type="imu">
+  	<xacro:macro name="gazebo" params="prefix:=">
+		<ros2_control name="GazeboSystem" type="system">
+			<hardware>
+				<plugin>gz_ros2_control/GazeboSimSystem</plugin>
+			</hardware>
+			<!-- <hardware>
+				<plugin>ign_ros2_control/IgnitionSystem</plugin>
+			</hardware> -->
+			<joint name="LF_HAA">
+				<command_interface name="effort"/>
+				<command_interface name="velocity" initial_value="0.0"/>
+				<state_interface name="position">
+					<param name="initial_value">0.0</param>
+				</state_interface>
+				<state_interface name="velocity"/>
+				<state_interface name="effort"/>
+			</joint>
+			<joint name="LF_HFE">
+				<command_interface name="effort"/>
+				<command_interface name="velocity" initial_value="0.0"/>
+				<state_interface name="position">
+					<param name="initial_value">0.72</param>
+				</state_interface>
+				<state_interface name="velocity"/>
+				<state_interface name="effort"/>
+			</joint>
+			<joint name="LF_KFE">
+				<command_interface name="effort"/>
+				<command_interface name="velocity" initial_value="0.0"/>
+				<state_interface name="position">
+					<param name="initial_value">-1.44</param>
+				</state_interface>
+				<state_interface name="velocity"/>
+				<state_interface name="effort"/>
+			</joint>
+			<joint name="LH_HAA">
+				<command_interface name="effort"/>
+				<command_interface name="velocity" initial_value="0.0"/>
+							<state_interface name="position">
+					<param name="initial_value">0.0</param>
+				</state_interface>
+				<state_interface name="velocity"/>
+				<state_interface name="effort"/>
+			</joint>
+			<joint name="LH_HFE">
+				<command_interface name="effort"/>
+				<command_interface name="velocity" initial_value="0.0"/>
+				<state_interface name="position">
+					<param name="initial_value">0.72</param>
+				</state_interface>
+				<state_interface name="velocity"/>
+				<state_interface name="effort"/>
+			</joint>
+			<joint name="LH_KFE">
+				<command_interface name="effort"/>
+				<command_interface name="velocity" initial_value="0.0"/>
+				<state_interface name="position">
+					<param name="initial_value">-1.44</param>
+				</state_interface>
+				<state_interface name="velocity"/>
+				<state_interface name="effort"/>
+			</joint>
+			<joint name="RF_HAA">
+				<command_interface name="effort"/>
+				<command_interface name="velocity" initial_value="0.0"/>
+				<state_interface name="position">
+					<param name="initial_value">0.0</param>
+				</state_interface>
+				<state_interface name="velocity"/>
+				<state_interface name="effort"/>
+			</joint>
+			<joint name="RF_HFE">
+				<command_interface name="effort"/>
+				<command_interface name="velocity" initial_value="0.0"/>
+				<state_interface name="position">
+					<param name="initial_value">0.72</param>
+				</state_interface>
+				<state_interface name="velocity"/>
+				<state_interface name="effort"/>
+			</joint>
+			<joint name="RF_KFE">
+				<command_interface name="effort"/>
+				<command_interface name="velocity" initial_value="0.0"/>
+				<state_interface name="position">
+					<param name="initial_value">-1.44</param>
+				</state_interface>
+				<state_interface name="velocity"/>
+				<state_interface name="effort"/>
+			</joint>
+			<joint name="RH_HAA">
+				<command_interface name="effort"/>
+				<command_interface name="velocity" initial_value="0.0"/>
+				<state_interface name="position">
+					<param name="initial_value">0.0</param>
+				</state_interface>
+				<state_interface name="velocity"/>
+				<state_interface name="effort"/>
+			</joint>
+			<joint name="RH_HFE">
+				<command_interface name="effort"/>
+				<command_interface name="velocity" initial_value="0.0"/>
+				<state_interface name="position">
+					<param name="initial_value">0.72</param>
+				</state_interface>
+				<state_interface name="velocity"/>
+				<state_interface name="effort"/>
+			</joint>
+			<joint name="RH_KFE">
+				<command_interface name="effort"/>
+				<command_interface name="velocity" initial_value="0.0"/>
+				<state_interface name="position">
+					<param name="initial_value">-1.44</param>
+				</state_interface>
+				<state_interface name="velocity"/>
+				<state_interface name="effort"/>
+			</joint>
+			<sensor name="imu_sensor">
+				<state_interface name="orientation.x"/>
+				<state_interface name="orientation.y"/>
+				<state_interface name="orientation.z"/>
+				<state_interface name="orientation.w"/>
+				<state_interface name="angular_velocity.x"/>
+				<state_interface name="angular_velocity.y"/>
+				<state_interface name="angular_velocity.z"/>
+				<state_interface name="linear_acceleration.x"/>
+				<state_interface name="linear_acceleration.y"/>
+				<state_interface name="linear_acceleration.z"/>
+			</sensor>
+		</ros2_control>
+		<gazebo>
+			<plugin filename="gz_ros2_control-system" name="gz_ros2_control::GazeboSimROS2ControlPlugin">
+				<parameters>$(find go1_description)/config/gazebo.yaml</parameters>
+			</plugin>
+			<plugin filename="gz-sim-imu-system"
+							name="gz::sim::systems::Imu">
+			</plugin>
+		</gazebo>
+		<gazebo reference="base">
+			<mu1>0.6</mu1>
+			<mu2>0.6</mu2>
+			<self_collide>1</self_collide>
+		</gazebo>
+		<gazebo>
+			<plugin name="gz::sim::systems::OdometryPublisher" filename="gz-sim-odometry-publisher-system">
+				<robot_base_frame>${prefix}base</robot_base_frame>
+				<dimensions>3</dimensions>
+			</plugin>
+		</gazebo>
+		<gazebo reference="imu_link">
+			<sensor name="imu_sensor" type="imu">
+				<always_on>1</always_on>
+				<update_rate>500</update_rate>
+				<visualize>true</visualize>
+				<topic>imu</topic>
+				<imu>
+					<angular_velocity>
+						<x>
+							<noise type="gaussian">
+								<mean>0.0</mean>
+								<stddev>2e-4</stddev>
+								<bias_mean>0.0000075</bias_mean>
+								<bias_stddev>0.0000008</bias_stddev>
+							</noise>
+						</x>
+						<y>
+							<noise type="gaussian">
+								<mean>0.0</mean>
+								<stddev>2e-4</stddev>
+								<bias_mean>0.0000075</bias_mean>
+								<bias_stddev>0.0000008</bias_stddev>
+							</noise>
+						</y>
+						<z>
+							<noise type="gaussian">
+								<mean>0.0</mean>
+								<stddev>2e-4</stddev>
+								<bias_mean>0.0000075</bias_mean>
+								<bias_stddev>0.0000008</bias_stddev>
+							</noise>
+						</z>
+					</angular_velocity>
+					<linear_acceleration>
+						<x>
+							<noise type="gaussian">
+								<mean>0.0</mean>
+								<stddev>1.7e-2</stddev>
+								<bias_mean>0.1</bias_mean>
+								<bias_stddev>0.001</bias_stddev>
+							</noise>
+						</x>
+						<y>
+							<noise type="gaussian">
+								<mean>0.0</mean>
+								<stddev>1.7e-2</stddev>
+								<bias_mean>0.1</bias_mean>
+								<bias_stddev>0.001</bias_stddev>
+							</noise>
+						</y>
+						<z>
+							<noise type="gaussian">
+								<mean>0.0</mean>
+								<stddev>1.7e-2</stddev>
+								<bias_mean>0.1</bias_mean>
+								<bias_stddev>0.001</bias_stddev>
+							</noise>
+						</z>
+					</linear_acceleration>
+				</imu>
+			</sensor>
+		</gazebo>
+		<gazebo reference="imu_joint">
+			<disableFixedJointLumping>true</disableFixedJointLumping>
+		</gazebo>
+		<gazebo reference="LF_foot_fixed">
+			<!-- Enable feedback for this joint -->
+			<provideFeedback>true</provideFeedback>
+			<!-- Prevent ros2_control from lumping this fixed joint with others -->
+			<disableFixedJointLumping>true</disableFixedJointLumping>
+			<sensor name="LF_ft_sensor" type="force_torque">
 			<always_on>1</always_on>
 			<update_rate>500</update_rate>
 			<visualize>true</visualize>
-			<topic>imu</topic>
-			<imu>
-				<angular_velocity>
-					<x>
-						<noise type="gaussian">
-							<mean>0.0</mean>
-							<stddev>2e-4</stddev>
-							<bias_mean>0.0000075</bias_mean>
-							<bias_stddev>0.0000008</bias_stddev>
-						</noise>
-					</x>
-					<y>
-						<noise type="gaussian">
-							<mean>0.0</mean>
-							<stddev>2e-4</stddev>
-							<bias_mean>0.0000075</bias_mean>
-							<bias_stddev>0.0000008</bias_stddev>
-						</noise>
-					</y>
-					<z>
-						<noise type="gaussian">
-							<mean>0.0</mean>
-							<stddev>2e-4</stddev>
-							<bias_mean>0.0000075</bias_mean>
-							<bias_stddev>0.0000008</bias_stddev>
-						</noise>
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
File: go1_description/xacro/robot.xacro (robot description, xacro)
@@ -153,3 +153,6 @@
 		<origin xyz="0.0 0.0 0.0" rpy="0.0 0.0 0.0"/>
 	</xacro:gps>
+	<xacro:if value="$(arg GAZEBO)">
+		<xacro:gazebo prefix="go1/"/>
+	</xacro:if>
 </robot>
